Commit message: Update ARM_STUDIO project

File: test piper/piper_assets/urdf/piper_description.urdf (robot description, URDF)
Before this commit: robot piper, 11 links, 10 joints
Links:
- link base_link: geometry collision mesh filename=../meshes/base_link.STL; visual box size=0.05 0.05 0.05
- link gripper_base: geometry collision mesh filename=../meshes/gripper_base.STL; visual box size=0.05 0.05 0.05
- link link1: geometry collision mesh filename=../meshes/link1.STL; visual box size=0.05 0.05 0.05
- link link2: geometry collision mesh filename=../meshes/link2.STL; visual box size=0.05 0.05 0.05
- link link3: geometry collision mesh filename=../meshes/link3.STL; visual box size=0.05 0.05 0.05
- link link4: geometry collision mesh filename=../meshes/link4.STL; visual box size=0.05 0.05 0.05
- link link5: geometry collision mesh filename=../meshes/link5.STL; visual box size=0.05 0.05 0.05
- link link6: geometry collision mesh filename=../meshes/link6.STL; visual box size=0.05 0.05 0.05
- link link7: geometry collision mesh filename=../meshes/link7.STL; visual box size=0.05 0.05 0.05
- link link8: geometry collision mesh filename=../meshes/link8.STL; visual box size=0.05 0.05 0.05
