Commit message: Sync local Arm_studio snapshot

File: robot/piper/piper_assets/urdf/piper_description_v100_camera.urdf (robot description, URDF)
Before this commit: robot piper_camera, 10 links, 9 joints
Links:
- link arm_base: geometry collision mesh filename=robot/piper/piper_assets/meshes/base_link.STL; visual mesh filename=robot/piper/piper_assets/meshes/dae/base_link.dae
- link link1: geometry collision mesh filename=robot/piper/piper_assets/meshes/link1.STL; visual mesh filename=robot/piper/piper_assets/meshes/dae/link1.dae
- link link2: geometry collision mesh filename=robot/piper/piper_assets/meshes/link2.STL; visual mesh filename=robot/piper/piper_assets/meshes/dae/link2.dae
- link link3: geometry collision mesh filename=robot/piper/piper_assets/meshes/link3.STL; visual mesh filename=robot/piper/piper_assets/meshes/dae/link3.dae
- link link4: geometry collision mesh filename=robot/piper/piper_assets/meshes/link4.STL; visual mesh filename=robot/piper/piper_assets/meshes/dae/link4.dae
- link link5: geometry collision mesh filename=robot/piper/piper_assets/meshes/link5.STL; visual mesh filename=robot/piper/piper_assets/meshes/dae/link5.dae
- link link6: geometry collision mesh filename=robot/piper/piper_assets/meshes/dae/camera_v3.dae; visual mesh filename=robot/piper/piper_assets/meshes/dae/camera_v3.dae
- link link7: geometry collision mesh filename=robot/piper/piper_assets/meshes/link7.STL; visual mesh filename=robot/piper/piper_assets/meshes/dae/link7.dae
- link link8: geometry collision mesh filename=robot/piper/piper_assets/meshes/link8.STL; visual mesh filename=robot/piper/piper_assets/meshes/dae/link8.dae
Joints:
- joint hand_camera_joint: origin xyz=0.0 0.075 0.03 rpy=0 -0.3 1.57  -> xyz=-0.075 0.0 0.035 rpy=0 -1.0472 0

File: robot/piper/piper_assets/urdf/piper_description_with_camera_left.xacro (robot description, xacro)
@@ -19,5 +19,5 @@
         <origin xyz="0 0 0" rpy="0 0 0" />
         <geometry>
-            <mesh filename="package://piper_description/meshes/dae/base_link.dae" />
+            <mesh filename="robot/piper/piper_assets/meshes/dae/base_link.dae" />
         </geometry>
         <material name="">
@@ -28,5 +28,5 @@
             <origin xyz="0 0 0" rpy="0 0 0" />
             <geometry>
-                <mesh filename="package://piper_description/meshes/base_link.STL" />
+                <mesh filename="robot/piper/piper_assets/meshes/base_link.STL" />
             </geometry>
         </collision>
@@ -49,5 +49,5 @@
         <origin xyz="0 0 0" rpy="0 0 0" />
         <geometry>
-            <mesh filename="package://piper_description/meshes/dae/link1.dae" />
+            <mesh filename="robot/piper/piper_assets/meshes/dae/link1.dae" />
         </geometry>
         <material name="">
@@ -58,5 +58,5 @@
             <origin xyz="0 0 0" rpy="0 0 1.5708" />
             <geometry>
-                <mesh filename="package://piper_description/meshes/link1.STL" />
+                <mesh filename="robot/piper/piper_assets/meshes/link1.STL" />
             </geometry>
         </collision>
@@ -86,5 +86,5 @@
         <origin xyz="0 0 0" rpy="0 0 0" />
         <geometry>
-            <mesh filename="package://piper_description/meshes/dae/link2.dae" />
+            <mesh filename="robot/piper/piper_assets/meshes/dae/link2.dae" />
         </geometry>
         <material name="">
@@ -95,5 +95,5 @@
             <origin xyz="0 0 0" rpy="0 0 0.1" />
             <geometry>
-                <mesh filename="package://piper_description/meshes/link2.STL" />
+                <mesh filename="robot/piper/piper_assets/meshes/link2.STL" />
             </geometry>
         </collision>
@@ -123,5 +123,5 @@
         <origin xyz="0 0 0" rpy="0 0 0" />
         <geometry>
-            <mesh filename="package://piper_description/meshes/dae/link3.dae" />
+            <mesh filename="robot/piper/piper_assets/meshes/dae/link3.dae" />
         </geometry>
         <material name="">
@@ -132,5 +132,5 @@
         <origin xyz="0 0 0" rpy="0 0 -1.75" />
         <geometry>
-            <mesh filename="package://piper_description/meshes/link3.STL" />
+            <mesh filename="robot/piper/piper_assets/meshes/link3.STL" />
         </geometry>
         </collision>
@@ -160,14 +160,14 @@
         <origin xyz="0 0 0" rpy="0 0 0" />
         <geometry>
-            <mesh filename="package://piper_description/meshes/dae/link4.dae" />
-        </geometry>
-        <material name="">
-            <color rgba="0.792156862745098 0.819607843137255 0.933333333333333 1" />
-        </material>
-        </visual>
-        <collision>
-        <origin xyz="0 0 0" rpy="0 0 0" />
-        <geometry>
-            <mesh filename="package://piper_description/meshes/link4.STL" />
+            <mesh filename="robot/piper/piper_assets/meshes/dae/link4.dae" />
+        </geometry>
+        <material name="">
+            <color rgba="0.792156862745098 0.819607843137255 0.933333333333333 1" />
+        </material>
+        </visual>
+        <collision>
+        <origin xyz="0 0 0" rpy="0 0 0" />
+        <geometry>
+            <mesh filename="robot/piper/piper_assets/meshes/link4.STL" />
         </geometry>
         </collision>
@@ -197,5 +197,5 @@
         <origin xyz="0 0 0" rpy="0 0 0" />
         <geometry>
-            <mesh filename="package://piper_description/meshes/dae/link5.dae" />
+            <mesh filename="robot/piper/piper_assets/meshes/dae/link5.dae" />
         </geometry>
         <material name="">
@@ -206,5 +206,5 @@
         <origin xyz="0 0 0" rpy="0 0 -3.14" />
         <geometry>
-            <mesh filename="package://piper_description/meshes/link5.STL" />
+            <mesh filename="robot/piper/piper_assets/meshes/link5.STL" />
         </geometry>
         </collision>
@@ -234,5 +234,5 @@
         <origin xyz="-0.002 -0.008 0" rpy="-1.57 0 0" />
         <geometry>
-            <mesh filename="package://piper_description/meshes/dae/camera_v3.dae"/>
+            <mesh filename="robot/piper/piper_assets/meshes/dae/camera_v3.dae"/>
         </geometry>
         <material name="">
@@ -243,5 +243,5 @@
         <origin xyz="-0.002 -0.008 0" rpy="-1.57 0 0" />
         <geometry>
-            <mesh filename="package://piper_description/meshes/dae/camera_v3.dae"/>
+            <mesh filename="robot/piper/piper_assets/meshes/dae/camera_v3.dae"/>
         </geometry>
         </collision>
@@ -271,5 +271,5 @@
         <origin xyz="0 0 0" rpy="0 0 0" />
         <geometry>
-            <mesh filename="package://piper_description/meshes/dae/link7.dae" />
+            <mesh filename="robot/piper/piper_assets/meshes/dae/link7.dae" />
         </geometry>
         <material name="">
@@ -280,5 +280,5 @@
         <origin xyz="-0.001 0 0.0003" rpy="0 3.14 0" />
         <geometry>
-            <mesh filename="package://piper_description/meshes/link7.STL" />
+            <mesh filename="robot/piper/piper_assets/meshes/link7.STL" />
         </geometry>
         </collision>
@@ -308,5 +308,5 @@
         <origin xyz="0 0 0" rpy="0 0 0" />
         <geometry>
-            <mesh filename="package://piper_description/meshes/dae/link8.dae" />
+            <mesh filename="robot/piper/piper_assets/meshes/dae/link8.dae" />
         </geometry>
         <material name="">
@@ -317,5 +317,5 @@
         <origin xyz="-0.001 0 0.0003" rpy="3.14 0 0" />
         <geometry>
-            <mesh filename="package://piper_description/meshes/link8.STL" />
+            <mesh filename="robot/piper/piper_assets/meshes/link8.STL" />
         </geometry>
         </collision>
@@ -328,4 +328,24 @@
         <limit lower="-0.05" upper="0" effort="100" velocity="1" />
     </joint>
+    <!-- Left wrist camera optical mount.  The sensor pose lives in this fixed
+         joint so ManiSkill can mount CameraConfig on hand_cam with identity pose. -->
+    <link name="${namespace}/hand_cam">
+        <inertial>
+            <origin xyz="0 0 0" rpy="0 0 0" />
+            <mass value="0.001" />
+            <inertia
+                ixx="1e-06"
+                ixy="0"
+                ixz="0"
+                iyy="1e-06"
+                iyz="0"
+                izz="1e-06" />
+        </inertial>
+    </link>
+    <joint name="${namespace}/hand_camera_joint" type="fixed">
+        <origin xyz="0.015040480 0.072650551 0.039562038" rpy="-0.052107272 -1.229275696 -1.516695972" />
+        <parent link="${namespace}/link6" />
+        <child link="${namespace}/hand_cam" />
+    </joint>
 </xacro:macro>
 </robot>

File: robot/piper/piper_assets/urdf/piper_description_with_camera_right.xacro (robot description, xacro)
@@ -19,5 +19,5 @@
         <origin xyz="0 0 0" rpy="0 0 0" />
         <geometry>
-            <mesh filename="package://piper_description/meshes/dae/base_link.dae" />
+            <mesh filename="robot/piper/piper_assets/meshes/dae/base_link.dae" />
         </geometry>
         <material name="">
@@ -28,5 +28,5 @@
             <origin xyz="0 0 0" rpy="0 0 0" />
             <geometry>
-                <mesh filename="package://piper_description/meshes/base_link.STL" />
+                <mesh filename="robot/piper/piper_assets/meshes/base_link.STL" />
             </geometry>
         </collision>
@@ -49,5 +49,5 @@
         <origin xyz="0 0 0" rpy="0 0 0" />
         <geometry>
-            <mesh filename="package://piper_description/meshes/dae/link1.dae" />
+            <mesh filename="robot/piper/piper_assets/meshes/dae/link1.dae" />
         </geometry>
         <material name="">
@@ -58,5 +58,5 @@
             <origin xyz="0 0 0" rpy="0 0 1.5708" />
             <geometry>
-                <mesh filename="package://piper_description/meshes/link1.STL" />
+                <mesh filename="robot/piper/piper_assets/meshes/link1.STL" />
             </geometry>
         </collision>
@@ -86,5 +86,5 @@
         <origin xyz="0 0 0" rpy="0 0 0" />
         <geometry>
-            <mesh filename="package://piper_description/meshes/dae/link2.dae" />
+            <mesh filename="robot/piper/piper_assets/meshes/dae/link2.dae" />
         </geometry>
         <material name="">
@@ -95,5 +95,5 @@
             <origin xyz="0 0 0" rpy="0 0 0.1" />
             <geometry>
-                <mesh filename="package://piper_description/meshes/link2.STL" />
+                <mesh filename="robot/piper/piper_assets/meshes/link2.STL" />
             </geometry>
         </collision>
@@ -123,5 +123,5 @@
         <origin xyz="0 0 0" rpy="0 0 0" />
         <geometry>
-            <mesh filename="package://piper_description/meshes/dae/link3.dae" />
+            <mesh filename="robot/piper/piper_assets/meshes/dae/link3.dae" />
         </geometry>
         <material name="">
@@ -132,5 +132,5 @@
         <origin xyz="0 0 0" rpy="0 0 -1.75" />
         <geometry>
-            <mesh filename="package://piper_description/meshes/link3.STL" />
+            <mesh filename="robot/piper/piper_assets/meshes/link3.STL" />
         </geometry>
         </collision>
@@ -160,14 +160,14 @@
         <origin xyz="0 0 0" rpy="0 0 0" />
         <geometry>
-            <mesh filename="package://piper_description/meshes/dae/link4.dae" />
-        </geometry>
-        <material name="">
-            <color rgba="0.792156862745098 0.819607843137255 0.933333333333333 1" />
-        </material>
-        </visual>
-        <collision>
-        <origin xyz="0 0 0" rpy="0 0 0" />
-        <geometry>
-            <mesh filename="package://piper_description/meshes/link4.STL" />
+            <mesh filename="robot/piper/piper_assets/meshes/dae/link4.dae" />
+        </geometry>
+        <material name="">
+            <color rgba="0.792156862745098 0.819607843137255 0.933333333333333 1" />
+        </material>
+        </visual>
+        <collision>
+        <origin xyz="0 0 0" rpy="0 0 0" />
+        <geometry>
+            <mesh filename="robot/piper/piper_assets/meshes/link4.STL" />
         </geometry>
         </collision>
@@ -197,5 +197,5 @@
         <origin xyz="0 0 0" rpy="0 0 0" />
         <geometry>
-            <mesh filename="package://piper_description/meshes/dae/link5.dae" />
+            <mesh filename="robot/piper/piper_assets/meshes/dae/link5.dae" />
         </geometry>
         <material name="">
@@ -206,5 +206,5 @@
         <origin xyz="0 0 0" rpy="0 0 -3.14" />
         <geometry>
-            <mesh filename="package://piper_description/meshes/link5.STL" />
+            <mesh filename="robot/piper/piper_assets/meshes/link5.STL" />
         </geometry>
         </collision>
@@ -234,5 +234,5 @@
         <origin xyz="-0.002 -0.008 0" rpy="-1.57 0 0" />
         <geometry>
-            <mesh filename="package://piper_description/meshes/dae/camera_v3.dae"/>
+            <mesh filename="robot/piper/piper_assets/meshes/dae/camera_v3.dae"/>
         </geometry>
         <material name="">
@@ -243,5 +243,5 @@
         <origin xyz="-0.002 -0.008 0" rpy="-1.57 0 0" />
         <geometry>
-            <mesh filename="package://piper_description/meshes/dae/camera_v3.dae"/>
+            <mesh filename="robot/piper/piper_assets/meshes/dae/camera_v3.dae"/>
         </geometry>
         </collision>
@@ -271,5 +271,5 @@
         <origin xyz="0 0 0" rpy="0 0 0" />
         <geometry>
-            <mesh filename="package://piper_description/meshes/dae/link7.dae" />
+            <mesh filename="robot/piper/piper_assets/meshes/dae/link7.dae" />
         </geometry>
         <material name="">
@@ -280,5 +280,5 @@
         <origin xyz="-0.001 0 0.0003" rpy="0 3.14 0" />
         <geometry>
-            <mesh filename="package://piper_description/meshes/link7.STL" />
+            <mesh filename="robot/piper/piper_assets/meshes/link7.STL" />
         </geometry>
         </collision>
@@ -308,5 +308,5 @@
         <origin xyz="0 0 0" rpy="0 0 0" />
         <geometry>
-            <mesh filename="package://piper_description/meshes/dae/link8.dae" />
+            <mesh filename="robot/piper/piper_assets/meshes/dae/link8.dae" />
         </geometry>
         <material name="">
@@ -317,5 +317,5 @@
         <origin xyz="-0.001 0 0.0003" rpy="3.14 0 0" />
         <geometry>
-            <mesh filename="package://piper_description/meshes/link8.STL" />
+            <mesh filename="robot/piper/piper_assets/meshes/link8.STL" />
         </geometry>
         </collision>
@@ -328,4 +328,24 @@
         <limit lower="-0.05" upper="0" effort="100" velocity="1" />
     </joint>
+    <!-- Right wrist camera optical mount.  The sensor pose lives in this fixed
+         joint so ManiSkill can mount CameraConfig on hand_cam with identity pose. -->
+    <link name="${namespace}/hand_cam">
+        <inertial>
+            <origin xyz="0 0 0" rpy="0 0 0" />
+            <mass value="0.001" />
+            <inertia
+                ixx="1e-06"
+                ixy="0"
+                ixz="0"
+                iyy="1e-06"
+                iyz="0"
+                izz="1e-06" />
+        </inertial>
+    </link>
+    <joint name="${namespace}/hand_camera_joint" type="fixed">
+        <origin xyz="0.013686479 0.069638234 0.038517091" rpy="0.010509198 -1.200507973 -1.583916315" />
+        <parent link="${namespace}/link6" />
+        <child link="${namespace}/hand_cam" />
+    </joint>
 </xacro:macro>
 </robot>
